File: pulse_stretcher/pulse_stretcher.kicad_sch (KiCad schematic)
At the start: 15 parts

Commit message: initial documentation and bom
Parts:
- removed R?: R_Small, symbol Device:R_Small
- added RV1: 150k, symbol Device:R_Potentiometer
- C1: renamed from C?; value C_Small -> 1uF
- C2: renamed from C?; value C_Small -> 10uF
- D1: renamed from D?; value LED -> pulse_indicator
- D2: renamed from D?; value LED -> on_indicator
- J2: renamed from J?; value Conn_Coaxial -> signal_out
- J3: renamed from J?; value Conn_Coaxial -> signal_in
- R1, R2: renamed from R?; value R_Small -> 10k
- R3, R4: renamed from R?; value R_Small -> 150
- gave numbers to parts that had none: 2
Connections:
- net at J2.1 (In): now also U1.13 (Q)
- net GND: now reaches J2.2 (Ext)
- net GND: now also J1.4 (GND), J1.5 (Shield), J3.2 (Ext), U1.1 (A), U1.8 (GND)
- net at R2.1: now also RV1.3
- net at R2.2: now also C1.1
- net at U1.14 (Cext): now also C1.2
- net at U1.15 (RCext): now also RV1.2
- net sign_input: now reaches U1.2 (B)
- net sign_input: now also J3.1 (In), U1.10 (B)
- net +5V: now reaches U1.3 (Clr)
- net +5V: now also U1.11 (Clr)
- net at D2.1 (K): now also U1.16 (VCC)
- net at D2.2 (A): now also R4.2
- net at J1.1 (VBUS): now also R4.1; no longer U1.16 (VCC)
- net at D1.1 (K): now also U1.9 (A)
- net at D1.2 (A): now also R3.2
- net at U1.5 (Q): now also R3.1
- net at U1.6 (Cext): now also C2.1
- net at U1.7 (RCext): now also R1.2
- net at R1.1: now also C2.2
- no-connect marks 2 -> 5
Other:
- moved on the sheet: C1, C2, D1, D2, J1, J2, J3, R1, R2, R3, R4, U1B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
