File: trigger_cable/trigger_cable.kicad_pcb (KiCad board)
At the start: 2 copper layers, 64 x 57.5 mm, 10 parts, among them J1 box_connector, J3 chn4, J4 chn3, J5 chn2, J6 chn1, J7 electrode_connector

Commit message: update board for production
Parts:
- added H1: MountingHole, MountingHole:MountingHole_3.2mm_M3, F.Cu at (61.0, 61.0)
- added H2: MountingHole, MountingHole:MountingHole_3.2mm_M3, F.Cu at (106.7, 61.0)
- added H3: MountingHole, MountingHole:MountingHole_3.2mm_M3, F.Cu at (61.0, 106.7)
- added H4: MountingHole, MountingHole:MountingHole_3.2mm_M3, F.Cu at (106.7, 106.7)
- J1: footprint Connector_Dsub:DSUB-37_Female_Horizontal_P2.77x2.54mm_EdgePinOffset9.40mm -> Connector_Dsub:DSUB-37_Male_Horizontal_P2.77x2.54mm_EdgePinOffset9.40mm
- moved J1 50.8 mm to (54.3, 59.1)
- moved J7 8.79 mm to (111.8, 59.3)
Routing:
- net Net-(J6-In): track 23.4 -> 100.9 mm
- net Net-(J5-In): track 41.7 -> 117.0 mm
- net Net-(J1-Pad5): track 67.9 -> 106.0 mm
- net Net-(J1-Pad6): track 62.0 -> 93.4 mm
- net Net-(J1-Pad7): track 50.9 -> 78.4 mm
- net Net-(J1-Pad8): track 44.4 -> 61.7 mm
- net Net-(J4-In): track 49.0 -> 34.1 mm
- net Net-(J3-In): track 60.5 -> 52.1 mm
Other:
- board size 64 x 57.5 mm -> 81.3 x 57.5 mm
