File: trigger_cable/trigger_cable.kicad_sch (KiCad schematic)
At the start: 10 parts, among them J1 DB37_Male, J2 DB25_Male, J3 chn4, J4 chn3, J5 chn2, J6 chn1

Commit message: first pcb version
Parts:
- removed J2: DB25_Male, symbol Connector:DB25_Male
- added J7: electrode_connector, Connector_Dsub:DSUB-37_Female_Horizontal_P2.77x2.54mm_EdgePinOffset9.40mm, symbol Connector:DB37_Male
- J1: value DB37_Male -> box_connector; footprint (none) -> Connector_Dsub:DSUB-37_Female_Horizontal_P2.77x2.54mm_EdgePinOffset9.40mm
- J3, J4, J5, J6: footprint (none) -> Connector_Coaxial:BNC_Amphenol_B6252HB-NPP3G-50_Horizontal
- R1, R2, R3, R4: footprint (none) -> Resistor_THT:R_Axial_DIN0309_L9.0mm_D3.2mm_P12.70mm_Horizontal
Connections:
- net GND: now also J7.10, J7.11, J7.12, J7.13, J7.14, J7.15, J7.16, J7.37, J7.9
- net at J1.5: now also J7.5
- net at J1.6: now also J7.6
- net at J1.7: now also J7.7
- net at J1.8: now also J7.8
- no-connect marks 33 -> 44

Commit message: update board for production
Parts:
- added H1, H2, H3, H4: MountingHole, MountingHole:MountingHole_3.2mm_M3, symbol Mechanical:MountingHole
- J1: footprint Connector_Dsub:DSUB-37_Female_Horizontal_P2.77x2.54mm_EdgePinOffset9.40mm -> Connector_Dsub:DSUB-37_Male_Horizontal_P2.77x2.54mm_EdgePinOffset9.40mm
Other:
- moved on the sheet: J6
